Commit message: modified:   urdf/disrobot_simple.urdf

File: urdf/disrobot_simple.urdf (robot description, URDF)
Before this commit: robot disrobot, 9 links, 8 joints
Links:
- added link base_footprint; visual box size=0.4572 0.4 0.00
Joints:
- added joint base_footprint_joint: type fixed, parent base_link, child base_footprint, origin xyz=0 0 0 rpy=0 0 0

Commit message: modified:   urdf/disrobot_simple.urdf

File: urdf/disrobot_simple.urdf (robot description, URDF)
Before this commit: robot disrobot, 10 links, 9 joints
Links:
- link base_footprint: geometry visual box size=0.61 0.4 0.00
